Commit message: ros trajectory control with arduino

File: rabota_description/urdf/rabota.URDF (robot description, URDF)
Before this commit: robot rabota, 5 links, 4 joints
Joints:
- removed joint link_1_Rot_joint
- removed joint link_2_Rot_joint
- added joint joint_1: type revolute, parent slider_link, child link_1, origin xyz=0 0 0 rpy=0 0 0, axis 0 0 1, limit lower=-1.57 upper=1.57 effort=1.5 velocity=8
- added joint joint_2: type revolute, parent link_1, child link_2, origin xyz=0.492 0 0 rpy=0 0 0, axis 0 0 1, limit lower=-1.57 upper=1.57 effort=1.5 velocity=8
- joint slider_pris_joint: type prismatic -> fixed

Commit message: control 3 motors throw joint trajectory action

File: rabota_description/urdf/rabota.URDF (robot description, URDF)
Before this commit: robot rabota, 5 links, 4 joints
Joints:
- removed joint slider_pris_joint
- added joint joint_3: type revolute, parent base_link, child slider_link, origin xyz=0.035 0 0.065 rpy=0 0 0, axis 0 0 1, limit lower=0 upper=0.6 effort=30 velocity=0.4
